File: VNTR-65.kicad_pcb (KiCad board)
At the start: 2 copper layers, 78 parts, among them U1 RP2350B, U10 SW_MX_HE, U11 SW_MX_HE, U12 SW_MX_HE, U13 SW_MX_HE, U14 SW_MX_HE, U15 SW_MX_HE, U16 SW_MX_HE, U17 SW_MX_HE, U18 SW_MX_HE, U19 SW_MX_HE, U2 NCP1117-3.3_SOT223, U20 SW_MX_HE, U21 SW_MX_HE, U22 SW_MX_HE, U23 SW_MX_HE, U24 SW_MX_HE, U25 SW_MX_HE, U26 SW_MX_HE, U27 SW_MX_HE, U28 SW_MX_HE, U29 SW_MX_HE, U3 W25Q128JVS, U30 SW_MX_HE, U31 SW_MX_HE, U32 SW_MX_HE, U33 SW_MX_HE, U34 SW_MX_HE, U35 SW_MX_HE, U36 SW_MX_HE, U37 SW_MX_HE, U38 SW_MX_HE, U39 SW_MX_HE, U4 USBLC6-2P6, U40 SW_MX_HE, U41 SW_MX_HE, U42 SW_MX_HE, U43 SW_MX_HE, U44 SW_MX_HE, U45 SW_MX_HE, U46 SW_MX_HE, U47 SW_MX_HE, U48 SW_MX_HE, U49 SW_MX_HE, U5 CD74HC4067M, U50 SW_MX_HE, U51 SW_MX_HE, U52 SW_MX_HE, U53 SW_MX_HE, U54 SW_MX_HE, U55 SW_MX_HE, U56 SW_MX_HE, U57 SW_MX_HE, U58 SW_MX_HE, U59 SW_MX_HE, U6 CD74HC4067M, U60 SW_MX_HE, U61 SW_MX_HE, U62 SW_MX_HE, U63 SW_MX_HE, U64 SW_MX_HE, U65 SW_MX_HE, U66 SW_MX_HE, U67 SW_MX_HE, U68 SW_MX_HE, U69 SW_MX_HE, U7 CD74HC4067M, U70 SW_MX_HE, U71 SW_MX_HE, U72 SW_MX_HE, U73 SW_MX_HE, U74 SW_MX_HE, U75 SW_MX_HE, U76 SW_MX_HE, U77 SW_MX_HE, U78 ER_OLEDM0.91_1x-I2C, U8 CD74HC4067M, U9 CD74HC4067M

Commit message: Assigned footprints to everything
Parts:
- added C1: 10u, Capacitor_SMD:C_0603_1608Metric, F.Cu at (56.5, 17.3)
- added C10: 100n, Capacitor_SMD:C_0603_1608Metric, F.Cu at (60.5, 17.3)
- added C11: 100n, Capacitor_SMD:C_0603_1608Metric, F.Cu at (60.5, 19.8)
- added C12: 100n, Capacitor_SMD:C_0603_1608Metric, F.Cu at (60.5, 22.3)
- added C13: 100n, Capacitor_SMD:C_0603_1608Metric, F.Cu at (60.5, 24.8)
- added C14: 100n, Capacitor_SMD:C_0603_1608Metric, F.Cu at (60.5, 27.3)
- added C15: 4.7u, Capacitor_SMD:C_0603_1608Metric, F.Cu at (60.5, 29.8)
- added C16: 100n, Capacitor_SMD:C_0603_1608Metric, F.Cu at (60.5, 32.3)
- added C17: 15p, Capacitor_SMD:C_0603_1608Metric, F.Cu at (60.5, 34.8)
- added C18: 15p, Capacitor_SMD:C_0603_1608Metric, F.Cu at (60.5, 37.3)
- added C19: 4.7u, Capacitor_SMD:C_0603_1608Metric, F.Cu at (64.5, 17.3)
- added C2: 10u, Capacitor_SMD:C_0603_1608Metric, F.Cu at (56.5, 19.8)
- added C20: 4.7u, Capacitor_SMD:C_0603_1608Metric, F.Cu at (64.5, 19.8)
- added C22: 100n, Capacitor_SMD:C_0603_1608Metric, F.Cu at (64.5, 22.3)
- added C23: 100n, Capacitor_SMD:C_0603_1608Metric, F.Cu at (64.5, 24.8)
- added C24: 100n, Capacitor_SMD:C_0603_1608Metric, F.Cu at (64.5, 27.3)
- added C25: 100n, Capacitor_SMD:C_0603_1608Metric, F.Cu at (64.5, 29.8)
- added C3: 100n, Capacitor_SMD:C_0603_1608Metric, F.Cu at (56.5, 22.3)
- added C4: 100n, Capacitor_SMD:C_0603_1608Metric, F.Cu at (56.5, 24.8)
- added C5: 4.7u, Capacitor_SMD:C_0603_1608Metric, F.Cu at (56.5, 27.3)
- added C6: 100n, Capacitor_SMD:C_0603_1608Metric, F.Cu at (56.5, 29.8)
- added C7: 100n, Capacitor_SMD:C_0603_1608Metric, F.Cu at (56.5, 32.3)
- added C8: 100n, Capacitor_SMD:C_0603_1608Metric, F.Cu at (56.5, 34.8)
- added C9: 100n, Capacitor_SMD:C_0603_1608Metric, F.Cu at (56.5, 37.3)
- added J1: Conn_01x03_Pin, Connector_USB:USB_C_Receptacle_HRO_TYPE-C-31-M-12, F.Cu at (124.0, 1.50)
- added J2: USB_C_Receptacle, Connector_PinHeader_2.54mm:PinHeader_1x03_P2.54mm_Vertical, F.Cu at (96.3, 8.77)
- added L1: 3.3u, Resistor_SMD:R_0603_1608Metric, F.Cu at (64.5, 32.3)
- added R1: 1k, Resistor_SMD:R_0603_1608Metric, F.Cu at (64.5, 34.8)
- added R10: 1k, Resistor_SMD:R_0603_1608Metric, F.Cu at (68.5, 32.3)
- added R11: 0, Resistor_SMD:R_0603_1608Metric, F.Cu at (68.5, 34.8)
- added R12: 1k, Resistor_SMD:R_0603_1608Metric, F.Cu at (68.5, 37.3)
- added R13: 10k, Resistor_SMD:R_0603_1608Metric, F.Cu at (72.5, 17.3)
- added R14: 10k, Resistor_SMD:R_0603_1608Metric, F.Cu at (72.5, 19.8)
- added R15: 1k, Resistor_SMD:R_0603_1608Metric, F.Cu at (72.5, 22.3)
- added R16: 4.7k, Resistor_SMD:R_0603_1608Metric, F.Cu at (72.5, 24.8)
- added R17: 4.7k, Resistor_SMD:R_0603_1608Metric, F.Cu at (72.5, 27.3)
- added R18: 1k, Resistor_SMD:R_0603_1608Metric, F.Cu at (72.5, 29.8)
- added R2: 10k, Resistor_SMD:R_0603_1608Metric, F.Cu at (64.5, 37.3)
- added R3: 5.1k, Resistor_SMD:R_0603_1608Metric, F.Cu at (68.5, 17.3)
- added R4: 5.1k, Resistor_SMD:R_0603_1608Metric, F.Cu at (68.5, 19.8)
- added R5: 33, Resistor_SMD:R_0603_1608Metric, F.Cu at (68.5, 22.3)
- added R6: 1k, Resistor_SMD:R_0603_1608Metric, F.Cu at (68.5, 24.8)
- added R8: 10k, Resistor_SMD:R_0603_1608Metric, F.Cu at (68.5, 27.3)
- added R9: DNF, Resistor_SMD:R_0603_1608Metric, F.Cu at (68.5, 29.8)
- added RV1: R_Potentiometer, PCM_Potentiometer_THT_AKL:Potentiometer_Bourns_PTA6043_Single_Slide, F.Cu at (1.74, 3.80)
- added SW1: SW_Push, Button_Switch_THT:SW_PUSH_6mm, F.Cu at (117.2, 32.2)
- added SW2: SW_Push, Button_Switch_THT:SW_PUSH_6mm, F.Cu at (97.5, 19.5)
- added SW3: RotaryEncoder, PCM_marbastlib-various:ROT_Alps_EC11E-Switch, F.Cu at (-22.0, 29.0)
- added Y1: Crystal_GND24, Crystal:Crystal_SMD_3225-4Pin_3.2x2.5mm, F.Cu at (101.3, 8.74)

Commit message: Positioned all the keys
Parts:
- moved U49 381.8 mm to (230.6, 32.4), turned to 90 degrees
- moved U48 364.0 mm to (213.1, 32.6), turned to 90 degrees
- moved U47 348.4 mm to (198.6, 32.4), turned to 90 degrees
- moved U46 333.0 mm to (184.6, 32.4), turned to 90 degrees
- moved U45 317.4 mm to (170.1, 32.6), turned to 90 degrees
- moved U25 302.1 mm to (155.4, 32.4), turned to 90 degrees
- moved U39 299.9 mm to (228.1, 18.1), turned to 90 degrees
- moved U44 287.3 mm to (141.4, 32.4), turned to 90 degrees
- moved U38 276.0 mm to (206.1, 18.1), turned to 90 degrees
- moved U24 272.6 mm to (127.5, 32.4), turned to 90 degrees
- moved U17 259.4 mm to (191.5, 17.9), turned to 90 degrees
- moved U23 258.0 mm to (113.0, 32.4), turned to 90 degrees
- moved U43 243.7 mm to (98.5, 32.4), turned to 90 degrees
- moved U37 242.9 mm to (177.1, 18.1), turned to 90 degrees
- moved U36 224.9 mm to (163.1, 18.1), turned to 90 degrees
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
Commit message: fix switch rotation
Parts:
- moved RV1 327.8 mm to (275.6, 83.8), turned to 90 degrees
- moved SW3 322.6 mm to (299.6, 3.00)
- moved U78 167.8 mm to (250.0, 6.31)
- turned U10 to 0 degrees
- turned U11 to 0 degrees
- turned U12 to 0 degrees
- turned U13 to 0 degrees
- turned U14 to 0 degrees
- turned U15 to 0 degrees
- turned U16 to 0 degrees
- turned U17 to 0 degrees
- turned U18 to 0 degrees
- turned U19 to 0 degrees
- turned U20 to 0 degrees
- turned U21 to 0 degrees
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
Commit message: moved components onto pcb and added pcb edge cut
Parts:
- J1: footprint Connector_USB:USB_C_Receptacle_HRO_TYPE-C-31-M-12 -> Connector_PinHeader_1.00mm:PinHeader_1x03_P1.00mm_Vertical_SMD_Pin1Left
- J2: footprint Connector_PinHeader_2.54mm:PinHeader_1x03_P2.54mm_Vertical -> Connector_USB:USB_C_Receptacle_HRO_TYPE-C-31-M-12
- moved C1 159.7 mm to (108.0, 104.4)
- moved C10 159.7 mm to (112.0, 104.4)
- moved C19 159.7 mm to (116.0, 104.4)
- moved R13 159.7 mm to (124.0, 104.4)
- moved R3 159.7 mm to (120.0, 104.4)
- moved C11 137.3 mm to (100.8, 87.5)
- moved C12 137.3 mm to (100.8, 90.0)
- moved C13 137.3 mm to (100.8, 92.5)
- moved C14 137.3 mm to (100.8, 95.0)
- moved C15 137.3 mm to (100.8, 97.5)
- moved C16 137.3 mm to (100.8, 100.0)
- moved C17 137.3 mm to (100.8, 102.5)
- moved C2 137.3 mm to (96.8, 87.5)
- moved C20 137.3 mm to (104.8, 87.5)
- moved C22 137.3 mm to (104.8, 90.0)
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Other:
- board outline added: 310 x 110 mm

Commit message: refine
Parts:
- moved R2 185.9 mm to (199.0, 19.0)
- moved R14 174.5 mm to (275.0, 23.0)
- moved C22 161.0 mm to (253.0, 27.0)
- moved C25 157.2 mm to (257.0, 58.0)
- moved R17 154.7 mm to (238.0, 4.00)
- moved R6 151.5 mm to (257.0, 61.0)
- moved C18 133.0 mm to (142.0, 18.0)
- moved L1 123.4 mm to (181.0, 3.00)
- moved U6 122.8 mm to (109.0, 14.0)
- moved C7 120.7 mm to (176.0, 9.00)
- moved R13 119.8 mm to (208.0, 19.0)
- moved C3 118.9 mm to (181.0, 6.00)
- moved C19 117.8 mm to (176.0, 3.00)
- moved C24 117.2 mm to (194.0, 19.0)
- moved C8 113.8 mm to (173.0, 18.0)
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