File: Hardware/PCB/VNTR-65.kicad_pcb (KiCad board)
At the start: 2 copper layers, 310 x 110 mm, 127 parts, among them J1 Conn_01x03_Pin, J2 USB_C_Receptacle, SW1 SW_Push, SW2 SW_Push, SW3 RotaryEncoder, U1 RP2350B, U10 SW_MX_HE, U11 SW_MX_HE, U12 SW_MX_HE, U13 SW_MX_HE, U14 SW_MX_HE, U15 SW_MX_HE, U16 SW_MX_HE, U17 SW_MX_HE, U18 SW_MX_HE, U19 SW_MX_HE, U2 NCP1117-3.3_SOT223, U20 SW_MX_HE, U21 SW_MX_HE, U22 SW_MX_HE, U23 SW_MX_HE, U24 SW_MX_HE, U25 SW_MX_HE, U26 SW_MX_HE, U27 SW_MX_HE, U28 SW_MX_HE, U29 SW_MX_HE, U3 W25Q128JVS, U30 SW_MX_HE, U31 SW_MX_HE, U32 SW_MX_HE, U33 SW_MX_HE, U34 SW_MX_HE, U35 SW_MX_HE, U36 SW_MX_HE, U37 SW_MX_HE, U38 SW_MX_HE, U39 SW_MX_HE, U4 USBLC6-2P6, U40 SW_MX_HE, U41 SW_MX_HE, U42 SW_MX_HE, U43 SW_MX_HE, U44 SW_MX_HE, U45 SW_MX_HE, U46 SW_MX_HE, U47 SW_MX_HE, U48 SW_MX_HE, U49 SW_MX_HE, U5 CD74HC4067M, U50 SW_MX_HE, U51 SW_MX_HE, U52 SW_MX_HE, U53 SW_MX_HE, U54 SW_MX_HE, U55 SW_MX_HE, U56 SW_MX_HE, U57 SW_MX_HE, U58 SW_MX_HE, U59 SW_MX_HE, U6 CD74HC4067M, U60 SW_MX_HE, U61 SW_MX_HE, U62 SW_MX_HE, U63 SW_MX_HE, U64 SW_MX_HE, U65 SW_MX_HE, U66 SW_MX_HE, U67 SW_MX_HE, U68 SW_MX_HE, U69 SW_MX_HE, U7 CD74HC4067M, U70 SW_MX_HE, U71 SW_MX_HE, U72 SW_MX_HE, U73 SW_MX_HE, U74 SW_MX_HE, U75 SW_MX_HE, U76 SW_MX_HE, U77 SW_MX_HE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

Commit message: Use KBPlacer to place keys in correct positions
Parts:
- moved U67 251.4 mm to (333.4, 95.2)
- moved U52 239.3 mm to (292.9, 76.2)
- moved U22 220.9 mm to (266.7, 38.1)
- moved U24 218.8 mm to (333.4, 38.1)
- moved R10 202.9 mm to (230.0, 129.0)
- moved SW1 198.0 mm to (219.0, 125.0)
- moved U23 195.2 mm to (295.3, 38.1)
- moved U53 187.7 mm to (333.4, 76.2)
- moved U21 187.5 mm to (247.7, 38.1)
- moved R12 186.4 mm to (230.0, 123.0)
- moved U19 182.9 mm to (209.6, 38.1)
- moved SW2 181.2 mm to (208.0, 125.0)
- moved R8 174.2 mm to (219.0, 120.0)
- moved C13 173.4 mm to (180.0, 129.0)
- moved R2 171.1 mm to (361.0, 74.0)
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Other:
- board size 310 x 110 mm -> 360 x 120 mm

Commit message: Worked on organising pcb
Parts:
- removed U77: SW_MX_HE, PCM_marbastlib-he:SW_MX_HE_0deg_1u
- C1, C10, C11, C12, C13, C14, C15, C16, C17, C18, C19, C2, C20, C22, C23, C24, C25, C3, C4, C5, C6, C7, C8, C9, R1, R10, R11, R12, R13, R14, R15, R16, R17, R18, R2, R3, R4, R5, R6, R8, R9: moved to B.Cu
- moved C13 125.2 mm to (266.0, 38.0)
- moved R13 121.0 mm to (205.0, 73.0)
- moved C20 121.0 mm to (85.0, 57.0)
- moved C14 116.0 mm to (216.0, 19.0)
- moved C16 101.6 mm to (285.0, 114.0)
- moved R6 100.0 mm to (238.0, 108.0)
- moved U5 98.9 mm to (146.0, 111.0), turned to 0 degrees
- moved U9 91.7 mm to (278.0, 79.0), turned to 0 degrees
- moved U6 87.3 mm to (183.0, 111.0), turned to 0 degrees
- moved C11 81.2 mm to (266.0, 114.0)
- moved C10 81.1 mm to (181.0, 45.0)
- moved C12 65.5 mm to (166.0, 76.0)
- moved L1 49.4 mm to (198.0, 126.0)
- moved C8 47.0 mm to (185.0, 76.0)
- moved C22 46.1 mm to (186.0, 108.0)
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Other:
- copper layers 2 -> 4
- board text added: "Main Sheet"
- board text added: "Switches"

Commit message: Routed PCB
Parts:
- C2, C22, C23, C24, C5, R10, R11, R18: moved to F.Cu
- moved C20 222.3 mm to (304.0, 95.0)
- moved R2 142.4 mm to (228.0, 20.0)
- moved R13 120.2 mm to (316.0, 27.0)
- moved SW1 114.5 mm to (176.0, 25.2)
- moved R6 113.5 mm to (335.0, 49.0)
- moved U3 112.7 mm to (220.5, 11.0)
- moved L1 108.9 mm to (227.0, 21.0)
- moved R9 108.5 mm to (226.0, 16.0)
- moved SW2 107.5 mm to (186.8, 25.2)
- moved R11 105.6 mm to (227.0, 16.0)
- moved C9 105.3 mm to (304.0, 114.0)
- moved C18 103.4 mm to (171.0, 26.0)
- moved R10 102.6 mm to (197.0, 18.0), turned to 180 degrees
- moved Y1 100.7 mm to (170.0, 28.0)
- moved C17 97.6 mm to (170.0, 29.0)
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Connections:
- R17 pad 2: unconnected-(R17-Pad2) -> +3.3V
- RV1 pad 1: +3V3 -> +3.3V
Routing:
- net +3.3V: track 0.00 -> 1341.2 mm, vias 0 -> 116
- net GND: track 0.00 -> 404.8 mm, vias 0 -> 42
- net GPIO4: track 0.00 -> 252.6 mm, vias 0 -> 20
- net GPIO1: track 0.00 -> 249.5 mm, vias 0 -> 25
- net GPIO3: track 0.00 -> 247.1 mm, vias 0 -> 24
- net GPIO2: track 0.00 -> 242.6 mm, vias 0 -> 18
- net Net-(U53-VOUT): track 0.00 -> 212.2 mm, vias 0 -> 10
- net Net-(U39-VOUT): track 0.00 -> 207.8 mm, vias 0 -> 6
- net Net-(U1-GPIO6): track 0.00 -> 205.2 mm, vias 0 -> 17
- net Net-(U24-VOUT): track 0.00 -> 193.0 mm, vias 0 -> 10
- net Net-(U38-VOUT): track 0.00 -> 180.3 mm, vias 0 -> 4
- net Net-(U52-VOUT): track 0.00 -> 172.1 mm, vias 0 -> 2
- net Net-(U37-VOUT): track 0.00 -> 164.0 mm, vias 0 -> 4
- net Net-(U68-VOUT): track 0.00 -> 158.2 mm, vias 0 -> 2
- net Net-(U67-VOUT): track 0.00 -> 152.9 mm
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- added copper zone on In2.Cu, net +3.3V
- added copper zone on In1.Cu, net GND
Other:
- board size 360 x 120 mm -> 400 x 150 mm
